File: hardware/Version_1.0/Version_1.0.kicad_sch (KiCad schematic)
At the start: 60 parts, among them J1 Conn_Coaxial, J2 Conn_Coaxial, J3 Conn_Coaxial, J4 Conn_Coaxial, J5 Conn_01x06_Pin, J6 Conn_01x06_Pin, J7 Conn_Coaxial, U1 ADF4351, Y1 SG-5032CAN

Commit message: edited the hardware v1.0
Parts:
- C1, C10, C11, C12, C13, C14, C15, C16, C17, C18, C19, C2, C20, C21, C22, C23, C24, C25, C26, C27, C28, C29, C3, C30, C31, C4, C5, C6, C7, C8, C9: footprint (none) -> Capacitor_SMD:C_0402_1005Metric
- D1: footprint (none) -> LED_SMD:LED_0402_1005Metric
- L1, L2, L3, L4, L5, L6, L7, L8: footprint (none) -> Inductor_SMD:L_0402_1005Metric
- R1, R10, R11, R2, R3, R4, R5, R6, R7, R8, R9: footprint (none) -> Resistor_SMD:R_0402_1005Metric
- U1: footprint Package_CSP:LFCSP-32-1EP_5x5mm_P0.5mm_EP3.25x3.25mm -> Ekene_Footprints:LFCSP-32-1EP_5x5mm_P0.5mm_EP3.1x3.1mm
Connections:
- net +3.3V: now also C12.2, C14.2, C19.2, C30.2
- net GND: now also J5.6 (Pin_6)
- no-connect marks 2 -> 1

Commit message: Finished v1 pcb
Parts:
- removed J1, J2: Conn_Coaxial, Connector_Coaxial:SMA_Molex_73251-1153_EdgeMount_Horizontal, symbol Connector:Conn_Coaxial
- removed J5, J6: Conn_01x06_Pin, Connector_PinSocket_2.54mm:PinSocket_1x06_P2.54mm_Vertical, symbol Connector:Conn_01x06_Pin
- added H1, H2: MountingHole_Pad, MountingHole:MountingHole_3.2mm_M3_Pad, symbol Mechanical:MountingHole_Pad
- added J1: Conn_02x05_Counter_Clockwise, Connector_PinHeader_2.54mm:PinHeader_2x05_P2.54mm_Vertical, symbol Connector_Generic:Conn_02x05_Counter_Clockwise
- added J5, J6: Conn_Coaxial, Connector_Coaxial:SMA_Molex_73251-1153_EdgeMount_Horizontal, symbol Connector:Conn_Coaxial
- renumbered J7 to J2
Connections:
- net +3.3V: now also J1.2 (Pin_2)
- net CE: now also J1.3 (Pin_3)
- net CLK: now also J1.7 (Pin_7)
- net CS: now also J1.5 (Pin_5)
- net GND: now also H1.1, H2.1, J1.1 (Pin_1), J1.4 (Pin_4), J5.2 (Ext), J6.2 (Ext)
- net LD: now also J1.9 (Pin_9)
- net MOSI: now also J1.6 (Pin_6)
- net MUXOUT: now also J1.8 (Pin_8)
- net PDB_RF: now also J1.10 (Pin_10)
- net OUTA+: no longer names the net of L1.2
- net OUTA+: now also J3.1 (In)
- net OUTA-: no longer names the net of L4.2
- net OUTA-: now also J4.1 (In); no longer J3.1 (In)
- net OUTB+: no longer names the net of L5.2
- net OUTB+: now also J5.1 (In)
- net OUTB-: no longer names the net of L8.2
- net OUTB-: now also J6.1 (In); no longer J4.1 (In)
Other:
- moved on the sheet: J2

Commit message: completed version 2 and version 3 pcb and production files completed
Other:
- title: ADF4351 Trial Board -> ADF4351
Changed lines of the file:
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@@
 	(paper "A4")
 	(title_block
-		(title "ADF4351 Trial Board")
+		(title "ADF4351")
 		(date "2026-07-21")
 		(rev "v1.0")
