File: hardware/Version_2.0/Version_2.0.kicad_pcb (KiCad board)
At the start: 4 copper layers, 40 x 33 mm, 50 parts, among them J1 Conn_02x05_Counter_Clockwise, J2 Conn_Coaxial, J3 Conn_Coaxial, J4 Conn_Coaxial, U1 ADF4351, Y1 SG-5032CAN

Commit message: updates
Other:
- board text added: "OUTA+"
- board text added: "OUTA-"
- board text added: "REFIN"
Changed lines of the file:
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@@
 		(layer "Edge.Cuts")
+	)
+	(gr_text "OUTA-"
+		(at 86.07 69.73 0)
+		(layer "F.SilkS")
+		(effects
+			(font
+				(size 1 1)
+				(thickness 0.25)
+				(bold yes)
+			)
+			(justify bottom)
+		)
+	)
+	(gr_text "OUTA+"
+		(at 86.1 53.07 0)
+		(layer "F.SilkS")
+		(effects
+			(font
+				(size 1 1)
+				(thickness 0.25)
+				(bold yes)
+			)
+			(justify bottom)
+		)
+	)
+	(gr_text "REFIN"
+		(at 109.9 58.47 0)
+		(layer "F.SilkS")
+		(effects
+			(font
+				(size 1 1)
+				(thickness 0.25)
+				(bold yes)
+			)
+			(justify bottom)
+		)
 	)
 	(gr_text "3v3"
